Commit message: Add files via upload

File: plane_bulldog.urdf (robot description, URDF)
Before this commit: robot colored_areas, 7 links, 6 joints
Links:
- link barrier_bottom: geometry collision box size=16 1 1; visual box size=16 1 1
- link barrier_left: geometry collision box size=1 16 1; visual box size=1 16 1
- link barrier_right: geometry collision box size=1 16 1; visual box size=1 16 1
- link barrier_top: geometry collision box size=16 1 1; visual box size=16 1 1
- link home_finish_area: geometry visual box size=2 14 0
- link home_start_area: geometry visual box size=2 14 0

Commit message: more tests done

File: plane_bulldog.urdf (robot description, URDF)
Before this commit: robot colored_areas, 7 links, 6 joints
Links:
- link barrier_bottom: geometry collision box size=14 1 1; visual box size=14 1 1
- link barrier_left: geometry collision box size=1 6 1; visual box size=1 6 1
- link barrier_right: geometry collision box size=1 6 1; visual box size=1 6 1
- link barrier_top: geometry collision box size=14 1 1; visual box size=14 1 1
- link home_finish_area: geometry visual box size=2 6 0
- link home_start_area: geometry visual box size=2 6 0
